File: pcb/bloo.kicad_pcb (KiCad board)
At the start: 2 copper layers, 84.9 x 94.9 mm, 107 parts, among them J1 Serial Debug Header, J10 Conn_01x06_Female, J4 Conn_ARM_JTAG_SWD_10, J5 SWD Header, J6 Conn_01x02_Female, J7 Conn_01x02_Female, J8 Conn_01x02_Female, J9 Conn_01x02_Female, M1 M1_Conn, M2 M2_Conn, M3 M1_Conn_Alt, M4 M2_Conn_Alt, Q0 Q_Photo_NPN, Q1 Q_Photo_NPN, Q10 Q_NMOS_GSD, Q11 Q_NMOS_GSD, Q12 Q_NMOS_GSD, Q2 Q_Photo_NPN, Q3 Q_Photo_NPN, Q4 Q_NMOS_SGD, Q5 Q_NMOS_SGD, Q6 Q_NMOS_SGD, Q7 Q_NMOS_SGD, Q8 Q_NMOS_SGD, Q9 Q_NMOS_GSD, SW1 SW, U1 YAAJ_BluePill_SWD_Breakout, U2 L293D, U3 LM1085-5.0, U4 APE8865Y5-33-HF-3

Commit message: update
Parts:
- removed J6, J7, J8, J9: Conn_01x02_Female, Connector_PinSocket_2.00mm:PinSocket_1x02_P2.00mm_Vertical
- removed Q4, Q5, Q6, Q7: Q_NMOS_SGD, Package_TO_SOT_THT:TO-92
- added C22: 0.1uF, Capacitor_SMD:C_1206_3216Metric_Pad1.33x1.80mm_HandSolder, F.Cu at (170.8, 95.2)
- added C5: 470nF, Capacitor_SMD:C_1206_3216Metric_Pad1.33x1.80mm_HandSolder, F.Cu at (167.0, 91.0)
- added C7: 10nF, Capacitor_SMD:C_1206_3216Metric_Pad1.33x1.80mm_HandSolder, F.Cu at (158.7, 94.1)
- added GYRO1: LY3200, custom_foot:LGA10, B.Cu at (160.0, 87.4)
- added JP5: Jumper_2_Open, Jumper:SolderJumper-2_P1.3mm_Bridged_Pad1.0x1.5mm, F.Cu at (173.0, 87.3)
- added L2: 10uH, Inductor_SMD:L_1206_3216Metric_Pad1.42x1.75mm_HandSolder, F.Cu at (168.2, 85.3)
- added R24: 10K, Resistor_SMD:R_1206_3216Metric_Pad1.30x1.75mm_HandSolder, F.Cu at (162.5, 94.0)
- Q8: footprint Package_TO_SOT_THT:TO-92 -> Package_TO_SOT_SMD:SOT-23; moved to B.Cu
- moved R17 2.88 mm to (142.9, 131.3)
- moved Q8 1.44 mm to (132.6, 62.2)
- moved C21 0.51 mm to (173.8, 137.7)
- moved Q1 0.22 mm to (169.9, 142.1)
- renumbered JP_SWO to JP1, JP_GND to JP2, JP_RST to JP3
Connections:
- U1 pad 16: Net-(U1-Pad16) -> BUZZER
- U1 pad 17: Net-(U1-Pad17) -> V_METER
- U1 pad 25: BUZZER -> GYRO_VREF
- U1 pad 26: V_METER -> GYRO_OUTZ
Routing:
- net BUZZER: track 77.2 -> 0.00 mm, vias 1 -> 0
- net GYRO_VREF: track 0.00 -> 60.2 mm, vias 0 -> 1
- net GYRO_OUTZ: track 0.00 -> 56.8 mm, vias 0 -> 1
- net M1_BACK: track 81.8 -> 28.3 mm
- net M2_FWD: track 95.8 -> 42.3 mm
- net GND: track 19.1 -> 62.3 mm, vias 180 -> 170
- net AGND2: track 0.00 -> 20.2 mm
- net AGND: track 94.3 -> 74.7 mm
- net Net-(C22-Pad1): track 0.00 -> 12.7 mm, vias 0 -> 2
- net RECEIV_4: track 38.4 -> 26.9 mm
- net RECEIV_2: track 39.3 -> 28.9 mm
- net RECEIV_1: track 26.2 -> 18.5 mm
- net EMIT_3: track 39.5 -> 34.8 mm, vias 1 -> 2
- net Net-(Q12-Pad3): track 6.37 -> 2.54 mm
- net RECEIV_3: track 28.9 -> 25.5 mm
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Other:
- board text added: "Jonathan Low v0.2 2023"
- board text removed: "Jonathan Low v0.1 2023"

Commit message: updates
Parts:
- removed J10: Conn_01x06_Female, Connector_PinSocket_2.54mm:PinSocket_1x06_P2.54mm_Vertical
- added J2: Conn_RST, Connector_PinSocket_2.54mm:PinSocket_1x01_P2.54mm_Vertical, F.Cu at (196.8, 117.9)
- added J3: BLE_PWR, Connector_PinSocket_2.54mm:PinSocket_1x01_P2.54mm_Vertical, F.Cu at (196.8, 105.0)
- added J6: BOOT0, Connector_PinSocket_2.54mm:PinSocket_1x01_P2.54mm_Vertical, F.Cu at (187.5, 102.7)
- added J7: BOOT0, Connector_PinSocket_2.54mm:PinSocket_1x01_P2.54mm_Vertical, F.Cu at (187.4, 106.6)
- added J8: Conn_01x04_Female, Connector_PinSocket_2.54mm:PinSocket_1x04_P2.54mm_Vertical, F.Cu at (196.8, 115.3)
- added JP6: Jumper_2_Open, Jumper:SolderJumper-2_P1.3mm_Open_Pad1.0x1.5mm, B.Cu at (193.0, 115.2)
- added Q4: Q_NMOS_GSD, Package_TO_SOT_SMD:SOT-23, B.Cu at (193.2, 111.5)
- added R25: 47k, Resistor_SMD:R_1206_3216Metric_Pad1.30x1.75mm_HandSolder, B.Cu at (193.0, 106.5)
- added R26: 47k, Resistor_SMD:R_1206_3216Metric_Pad1.30x1.75mm_HandSolder, F.Cu at (184.4, 104.4)
- C5, C7, JP5, R24: moved to B.Cu
- moved R17 65.6 mm to (132.6, 66.5), turned to 90 degrees
- moved JP5 18.5 mm to (155.7, 93.9), turned to 90 degrees
- moved C22 10.5 mm to (165.0, 86.5)
- moved R24 3.92 mm to (158.6, 94.5)
- moved C7 2.97 mm to (161.7, 94.1), turned to 90 degrees
- moved C5 2.29 mm to (164.8, 91.7)
- moved R11 1.07 mm to (130.5, 57.5)
Routing:
- net BUZZER: track 0.00 -> 58.5 mm
- net M1_BACK: track 28.3 -> 80.2 mm
- net GND: track 62.3 -> 14.2 mm, vias 170 -> 164
- net M2_FWD: track 42.3 -> 90.3 mm
- net +3V3: track 263.6 -> 292.7 mm, vias 4 -> 8
- net RST: track 69.2 -> 95.0 mm
- net AGND2: track 20.2 -> 32.8 mm, vias 0 -> 1
- net Net-(C5-Pad1): track 3.17 -> 15.2 mm, vias 1 -> 2
- net V_METER: track 13.6 -> 23.5 mm
- net Net-(J3-Pad1): track 0.00 -> 8.03 mm
- net Net-(C5-Pad2): track 0.00 -> 7.60 mm
- net Net-(J8-Pad3): track 0.00 -> 7.49 mm
- net Net-(J6-Pad1): track 0.00 -> 7.08 mm
- net BUTTON: track 81.6 -> 82.8 mm
- net EMIT_1: vias 1 -> 2

Commit message: updates
Routing:
- net GND: track 14.2 -> 23.9 mm, vias 164 -> 215
- net +3V3: track 292.7 -> 289.7 mm
- net SWDCLK: track 45.8 -> 44.0 mm
- net Net-(J4-Pad6): track 14.1 -> 13.1 mm
- net BUTTON: track 82.8 -> 83.7 mm

Commit message: v0.2?
Parts:
- C22, L2: moved to B.Cu
- moved L2 5.36 mm to (170.4, 90.2)
- moved C22 2.22 mm to (166.4, 88.2), turned to 135 degrees
- moved C5 2.19 mm to (164.5, 93.9)
Routing:
- net Net-(C22-Pad1): track 12.7 -> 18.1 mm, vias 2 -> 3
- net +3V3: track 289.7 -> 294.5 mm, vias 8 -> 9
- net Net-(C5-Pad1): track 15.2 -> 10.9 mm
- net AGND2: track 32.8 -> 36.6 mm, vias 1 -> 0
- net M1_ENC_B: track 88.4 -> 87.4 mm
- net M1_ENC_A: track 91.5 -> 90.5 mm
- net GND: vias 215 -> 221
Other:
- board text added: "User Spacers For Screw"
