File: pcb/bloo copy.sch (KiCad schematic (older format))
At the start: 106 parts, among them J1 Serial Debug Header, J10 Conn_01x06_Female, J4 Conn_ARM_JTAG_SWD_10, J5 SWD Header, M1 M1_Conn, M2 M2_Conn, M3 M1_Conn_Alt, M4 M2_Conn_Alt, Q0 Q_Photo_NPN, Q1 Q_Photo_NPN, Q10 Q_NMOS_GSD, Q11 Q_NMOS_GSD, Q12 Q_NMOS_GSD, Q2 Q_Photo_NPN, Q3 Q_Photo_NPN, Q8 Q_NMOS_SGD, Q9 Q_NMOS_GSD, SW1 SW, U1 YAAJ_BluePill_SWD_Breakout, U2 L293D, U3 LM1085-5.0, U4 APE8865Y5-33-HF-3

Commit message: updates
Parts:
- removed J10: Conn_01x06_Female, Connector_PinSocket_2.54mm:PinSocket_1x06_P2.54mm_Vertical, symbol Connector:Conn_01x06_Female
- added J2: Conn_RST, Connector_PinSocket_2.54mm:PinSocket_1x01_P2.54mm_Vertical, symbol Connector:Conn_01x01_Female
- added J3: BLE_PWR, Connector_PinSocket_2.54mm:PinSocket_1x01_P2.54mm_Vertical, symbol Connector:Conn_01x01_Female
- added J6, J7: BOOT0, Connector_PinSocket_2.54mm:PinSocket_1x01_P2.54mm_Vertical, symbol Connector:Conn_01x01_Female
- added J8: Conn_01x04_Female, Connector_PinSocket_2.54mm:PinSocket_1x04_P2.54mm_Vertical, symbol Connector:Conn_01x04_Female
- added JP6: Jumper_2_Open, Jumper:SolderJumper-2_P1.3mm_Open_Pad1.0x1.5mm, symbol Jumper:Jumper_2_Open
- added Q4: Q_NMOS_GSD, Package_TO_SOT_SMD:SOT-23, symbol Device:Q_NMOS_GSD
- added R25, R26: 47k, Resistor_SMD:R_1206_3216Metric_Pad1.30x1.75mm_HandSolder, symbol bloo-rescue:R-Device-mouse_v2-rescue
Connections:
- net +3V3: now also R25.1
- net +5V: now also J8.4 (Pin_4)
- net GND: now also JP6.2 (B), Q4.2 (S), R26.1
- net RST: now also J2.1 (Pin_1)
- net at C6.1, FB4.1, J1.2 (Pin_2): now also J8.1 (Pin_1)
- net at C8.1, FB3.2, J1.3 (Pin_3): now also J8.2 (Pin_2)
- new net: J8.3 (Pin_3), JP6.1 (A), Q4.3 (D)
- new net: J3.1 (Pin_1), Q4.1 (G), R25.2
- new net: J6.1 (Pin_1), J7.1 (Pin_1), R26.2
- no-connect marks 15 -> 13
Changed lines of the file:
@@
 	14450 7825 14600 7825
-Wire Wire Line
-	11750 8075 12825 8075
-Wire Wire Line
-	11750 7975 12650 7975
 Wire Wire Line
 	13875 8300 13875 7975
@@
 	3900 7575 4275 7575
 $Comp
-L Connector:Conn_01x06_Female J10
-U 1 1 64870CA0
-P 11500 9325
-F 0 "J10" H 11392 8800 50  0000 C CNN
-F 1 "Conn_01x06_Female" H 11392 8891 50  0000 C CNN
-F 2 "Connector_PinSocket_2.54mm:PinSocket_1x06_P2.54mm_Vertical" H 11500 9325 50  0001 C CNN
-F 3 "~" H 11500 9325 50  0001 C CNN
-	1    11500 9325
-	-1   0    0    1
-$EndComp
-Wire Wire Line
-	11700 9425 12825 9425
-Wire Wire Line
-	12825 9425 12825 8075
-Connection ~ 12825 8075
-Wire Wire Line
-	12825 8075 13475 8075
-Wire Wire Line
-	11700 9325 12650 9325
-Wire Wire Line
-	12650 9325 12650 7975
-Connection ~ 12650 7975
-Wire Wire Line
-	12650 7975 13875 7975
-Wire Wire Line
-	11700 9125 12250 9125
-Wire Wire Line
-	12250 9125 12250 8800
-Wire Wire Line
-	11700 9225 12250 9225
-Wire Wire Line
-	12250 9225 12250 9650
-$Comp
 L power:GND #PWR0118
 U 1 1 64919533
-P 12250 9650
-F 0 "#PWR0118" H 12250 9400 50  0001 C CNN
-F 1 "GND" H 12255 9477 50  0000 C CNN
-F 2 "" H 12250 9650 50  0001 C CNN
-F 3 "" H 12250 9650 50  0001 C CNN
-	1    12250 9650
-	1    0    0    -1
-$EndComp
-NoConn ~ 11700 9025
-NoConn ~ 11700 9525
+P 11550 10225
+F 0 "#PWR0118" H 11550 9975 50  0001 C CNN
+F 1 "GND" H 11555 10052 50  0000 C CNN
+F 2 "" H 11550 10225 50  0001 C CNN
+F 3 "" H 11550 10225 50  0001 C CNN
+	1    11550 10225
+	1    0    0    -1
+$EndComp
 $Comp
 L power:+5V #PWR0117
 U 1 1 649E8DEB
-P 12250 8800
-F 0 "#PWR0117" H 12250 8650 50  0001 C CNN
-F 1 "+5V" H 12265 8973 50  0000 C CNN
-F 2 "" H 12250 8800 50  0001 C CNN
-F 3 "" H 12250 8800 50  0001 C CNN
-	1    12250 8800
+P 12250 8575
+F 0 "#PWR0117" H 12250 8425 50  0001 C CNN
+F 1 "+5V" H 12265 8748 50  0000 C CNN
+F 2 "" H 12250 8575 50  0001 C CNN
+F 3 "" H 12250 8575 50  0001 C CNN
+	1    12250 8575
 	1    0    0    -1
 $EndComp
@@
 Wire Wire Line
 	13100 6025 13900 6025
+$Comp
+L Device:Q_NMOS_GSD Q4
+U 1 1 645924B5
+P 11450 9800
+F 0 "Q4" H 11654 9846 50  0000 L CNN
+F 1 "Q_NMOS_GSD" H 11654 9755 50  0000 L CNN
+F 2 "Package_TO_SOT_SMD:SOT-23" H 11650 9900 50  0001 C CNN
+F 3 "~" H 11450 9800 50  0001 C CNN
+	1    11450 9800
+	1    0    0    -1
+$EndComp
+$Comp
+L Jumper:Jumper_2_Open JP6
+U 1 1 645A07DA
+P 11600 9300
+F 0 "JP6" H 11600 9535 50  0000 C CNN
+F 1 "Jumper_2_Open" H 11600 9444 50  0000 C CNN
+F 2 "Jumper:SolderJumper-2_P1.3mm_Open_Pad1.0x1.5mm" H 11600 9300 50  0001 C CNN
+F 3 "~" H 11600 9300 50  0001 C CNN
+	1    11600 9300
+	1    0    0    -1
+$EndComp
+Wire Wire Line
+	12250 8575 12250 8700
+Wire Wire Line
+	11000 8700 12250 8700
+Wire Wire Line
+	11000 8900 12650 8900
+Wire Wire Line
+	11000 9000 12825 9000
+Wire Wire Line
+	11000 8800 11150 8800
+Wire Wire Line
+	11150 8800 11150 9300
+Wire Wire Line
+	11400 9300 11300 9300
+$Comp
+L power:GND #PWR0133
+U 1 1 64A2557E
+P 11875 9400
+F 0 "#PWR0133" H 11875 9150 50  0001 C CNN
+F 1 "GND" H 11880 9227 50  0000 C CNN
+F 2 "" H 11875 9400 50  0001 C CNN
+F 3 "" H 11875 9400 50  0001 C CNN
+	1    11875 9400
+	1    0    0    -1
+$EndComp
+Wire Wire Line
+	11875 9400 11875 9300
+Wire Wire Line
+	11875 9300 11800 9300
+Wire Wire Line
+	11550 10000 11550 10225
+Wire Wire Line
+	11300 9300 11300 9600
+Wire Wire Line
+	11300 9600 11550 9600
+Connection ~ 11300 9300
+Wire Wire Line
+	11300 9300 11150 9300
+$Comp
+L Connector:Conn_01x01_Female J3
+U 1 1 64B49AC8
+P 10650 9475
+F 0 "J3" V 10588 9387 50  0000 R CNN
+F 1 "BLE_PWR" V 10750 9575 50  0000 R CNN
+F 2 "Connector_PinSocket_2.54mm:PinSocket_1x01_P2.54mm_Vertical" H 10650 9475 50  0001 C CNN
+F 3 "~" H 10650 9475 50  0001 C CNN
+	1    10650 9475
+	0    -1   -1   0
+$EndComp
+Wire Wire Line
+	10650 9800 10650 9675
+$Comp
+L bloo-rescue:R-Device-mouse_v2-rescue R25
+U 1 1 64BDD530
+P 11000 9650
+F 0 "R25" V 10793 9650 50  0000 C CNN
+F 1 "47k" V 10884 9650 50  0000 C CNN
+F 2 "Resistor_SMD:R_1206_3216Metric_Pad1.30x1.75mm_HandSolder" V 10930 9650 50  0001 C CNN
+F 3 "~" H 11000 9650 50  0001 C CNN
+	1    11000 9650
+	1    0    0    -1
+$EndComp
+Wire Wire Line
+	12650 7975 13875 7975
+Wire Wire Line
+	11750 7975 12650 7975
+Connection ~ 12650 7975
+Wire Wire Line
+	12650 8900 12650 7975
+Wire Wire Line
+	12825 8075 13475 8075
+Wire Wire Line
+	11750 8075 12825 8075
+Connection ~ 12825 8075
+Wire Wire Line
+	12825 9000 12825 8075
+Wire Wire Line
+	11250 9800 11000 9800
+Connection ~ 11000 9800
+Wire Wire Line
+	11000 9800 10650 9800
+$Comp
+L power:+3V3 #PWR0134
+U 1 1 64E92ADF
+P 11000 9500
+F 0 "#PWR0134" H 11000 9350 50  0001 C CNN
+F 1 "+3V3" H 11015 9673 50  0000 C CNN
+F 2 "" H 11000 9500 50  0001 C CNN
+F 3 "" H 11000 9500 50  0001 C CNN
+	1    11000 9500
+	1    0    0    -1
+$EndComp
+$Comp
+L Connector:Conn_01x01_Female J2
+U 1 1 64E97D51
+P 7275 5600
+F 0 "J2" H 7303 5626 50  0000 L CNN
+F 1 "Conn_RST" H 7303 5535 50  0000 L CNN
+F 2 "Connector_PinSocket_2.54mm:PinSocket_1x01_P2.54mm_Vertical" H 7275 5600 50  0001 C CNN
+F 3 "~" H 7275 5600 50  0001 C CNN
+	1    7275 5600
+	-1   0    0    1
+$EndComp
+Text GLabel 7625 5600 2    50   Input ~ 0
+RST
+Wire Wire Line
+	7625 5600 7475 5600
+$Comp
+L Connector:Conn_01x01_Female J7
+U 1 1 64EE258E
+P 7450 4400
+F 0 "J7" V 7388 4312 50  0000 R CNN
+F 1 "BOOT0" V 7550 4500 50  0000 R CNN
+F 2 "Connector_PinSocket_2.54mm:PinSocket_1x01_P2.54mm_Vertical" H 7450 4400 50  0001 C CNN
+F 3 "~" H 7450 4400 50  0001 C CNN
+	1    7450 4400
+	0    -1   -1   0
+$EndComp
+Wire Wire Line
+	7450 4725 7450 4600
+$Comp
+L bloo-rescue:R-Device-mouse_v2-rescue R26
+U 1 1 64EE2599
+P 7950 4725
+F 0 "R26" V 7743 4725 50  0000 C CNN
+F 1 "47k" V 7834 4725 50  0000 C CNN
+F 2 "Resistor_SMD:R_1206_3216Metric_Pad1.30x1.75mm_HandSolder" V 7880 4725 50  0001 C CNN
+F 3 "~" H 7950 4725 50  0001 C CNN
+	1    7950 4725
+	0    1    1    0
+$EndComp
+Wire Wire Line
+	7800 4725 7450 4725
+$Comp
+L Connector:Conn_01x01_Female J6
+U 1 1 64FAD9B6
+P 7150 4400
+F 0 "J6" V 7088 4312 50  0000 R CNN
+F 1 "BOOT0" V 7250 4500 50  0000 R CNN
+F 2 "Connector_PinSocket_2.54mm:PinSocket_1x01_P2.54mm_Vertical" H 7150 4400 50  0001 C CNN
+F 3 "~" H 7150 4400 50  0001 C CNN
+	1    7150 4400
+	0    -1   -1   0
+$EndComp
+$Comp
+L power:GND #PWR0152
+U 1 1 64FB1FED
+P 8275 4825
+F 0 "#PWR0152" H 8275 4575 50  0001 C CNN
+F 1 "GND" H 8280 4652 50  0000 C CNN
+F 2 "" H 8275 4825 50  0001 C CNN
+F 3 "" H 8275 4825 50  0001 C CNN
+	1    8275 4825
+	1    0    0    -1
+$EndComp
+Wire Wire Line
+	8275 4825 8275 4725
+Wire Wire Line
+	8275 4725 8100 4725
+Wire Wire Line
+	7450 4725 7150 4725
+Wire Wire Line
+	7150 4725 7150 4600
+Connection ~ 7450 4725
+$Comp
+L Connector:Conn_01x04_Female J8
+U 1 1 64546237
+P 10800 8900
+F 0 "J8" H 10692 8475 50  0000 C CNN
+F 1 "Conn_01x04_Female" H 10692 8566 50  0000 C CNN
+F 2 "Connector_PinSocket_2.54mm:PinSocket_1x04_P2.54mm_Vertical" H 10800 8900 50  0001 C CNN
+F 3 "~" H 10800 8900 50  0001 C CNN
+	1    10800 8900
+	-1   0    0    1
+$EndComp
 $EndSCHEMATC
